File: elec/layout/default/lis3mdltr.kicad_pcb (KiCad board)
At the start: 2 copper layers, 225.7 x 100.8 mm, 0 parts

Commit message: initial layout
Parts:
- added C1: Multilayer Ceramic Capacitors MLCC - SMD/SMT 100nF 10V 0402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, lib:C0402, F.Cu at (158.1, 98.9)
- added C2: Multilayer Ceramic Capacitors MLCC - SMD/SMT 1uF 6.3V 0402 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, lib:C0402, F.Cu at (158.1, 97.9)
- added C3: Multilayer Ceramic Capacitors MLCC - SMD/SMT 100nF 10V 0402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, lib:C0402, F.Cu at (154.4, 95.8)
- added R1: Chip Resistor - Surface Mount 1.1KOhms ±5% 1/16W 0402 RoHS, lib:R0402, F.Cu at (155.4, 95.8)
- added U1: , lib:LGA-12_L2.0-W2.0-P0.50-BL, F.Cu at (155.6, 98.2)
Routing:
- net gnd: track 0.00 -> 6.35 mm
- net vcc: track 0.00 -> 3.66 mm
- net c1: track 0.00 -> 1.40 mm
- net miso: track 0.00 -> 1.04 mm
