File: elec/layout/default/lis3mdltr.kicad_pcb (KiCad board)
At the start: 2 copper layers, 225.7 x 100.8 mm, 5 parts

Commit message: updating layout
Parts:
- C1, C3: value Multilayer Ceramic Capacitors MLCC - SMD/SMT 100nF 10V 0402 RoHS -> 16V 100nF X7R ±10% 0402 Multilayer Ceramic Capacitors MLCC - SMD/SMT ROHS
- C2: value Multilayer Ceramic Capacitors MLCC - SMD/SMT 1uF 6.3V 0402 RoHS -> 25V 1uF X5R ±10% 0402 Multilayer Ceramic Capacitors MLCC - SMD/SMT ROHS
- R1: value Chip Resistor - Surface Mount 1.1KOhms ±5% 1/16W 0402 RoHS -> 62.5mW Thick Film Resistors ±100ppm/℃ ±1% 1kΩ 0402 Chip Resistor - Surface Mount ROHS
Changed lines of the file:
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@@
         (effects (font (size 1 1) (thickness 0.15)))
     )
-    (fp_text value "Multilayer Ceramic Capacitors MLCC - SMD/SMT 100nF 10V 0402 RoHS" (at 0 1.16) (layer "F.Fab")
+    (fp_text value "16V 100nF X7R ±10% 0402  Multilayer Ceramic Capacitors MLCC - SMD/SMT ROHS" (at 0 1.16) (layer "F.Fab")
         (effects (font (size 1 1) (thickness 0.15)))
     )
@@
         (effects (font (size 1 1) (thickness 0.15)))
     )
-    (fp_text value "Multilayer Ceramic Capacitors MLCC - SMD/SMT 100nF 10V 0402 RoHS" (at 0 1.16 90) (layer "F.Fab")
+    (fp_text value "16V 100nF X7R ±10% 0402  Multilayer Ceramic Capacitors MLCC - SMD/SMT ROHS" (at 0 1.16 90) (layer "F.Fab")
         (effects (font (size 1 1) (thickness 0.15)))
     )
@@
         (effects (font (size 1 1) (thickness 0.15)))
     )
-    (fp_text value "Multilayer Ceramic Capacitors MLCC - SMD/SMT 1uF 6.3V 0402 RoHS" (at 0 1.16) (layer "F.Fab")
+    (fp_text value "25V 1uF X5R ±10% 0402  Multilayer Ceramic Capacitors MLCC - SMD/SMT ROHS" (at 0 1.16) (layer "F.Fab")
         (effects (font (size 1 1) (thickness 0.15)))
     )
@@
         (effects (font (size 1 1) (thickness 0.15)))
     )
-    (fp_text value "Chip Resistor - Surface Mount 1.1KOhms ±5% 1/16W 0402 RoHS" (at 0 1.17 90) (layer "F.Fab")
-        (effects (font (size 1 1) (thickness 0.15)))
-    )
+    (fp_text value "62.5mW Thick Film Resistors ±100ppm/℃ ±1% 1kΩ 0402  Chip Resistor - Surface Mount ROHS" (at 0 1.17 90) (layer "F.Fab")
+        (effects (font (size 1 1) (thickness 0.15)))
+    )
